File: RX_Ant.kicad_pcb (KiCad board)
At the start: 2 copper layers, 100 x 100 mm, 2528 parts, among them J1 CONN_COAXIAL, J10 CONN_COAXIAL, J11 CONN_01X06, J12 CONN_01X05, J13 CONN_COAXIAL, J14 CONN_COAXIAL, J15 CONN_COAXIAL, J16 CONN_01X01, J17 CONN_01X01, J18 CONN_01X01, J19 CONN_01X01, J2 CONN_COAXIAL, J20 CONN_01X01, J21 CONN_01X01, J22 CONN_01X01, J23 CONN_01X01, J24 CONN_COAXIAL, J25 CONN_COAXIAL, J26 CONN_COAXIAL, J27 CONN_COAXIAL, J28 CONN_COAXIAL, J29 CONN_COAXIAL, J3 CONN_COAXIAL, J30 CONN_COAXIAL, J31 CONN_COAXIAL, J32 CONN_COAXIAL, J33 CONN_COAXIAL, J34 CONN_COAXIAL, J35 CONN_COAXIAL, J36 CONN_COAXIAL, J4 CONN_COAXIAL, J5 CONN_COAXIAL, J6 CONN_COAXIAL, J7 CONN_COAXIAL, J8 CONN_COAXIAL, J9 CONN_COAXIAL

Commit message: new routing, new gerber
Parts:
- removed the REF** at (59.0, 71.0) (x3)
- removed the REF** at (58.0, 71.0) (x3)
- removed the REF** at (57.0, 71.0) (x3)
- removed the REF** at (56.0, 71.0) (x3)
- removed the REF** at (55.0, 71.0) (x3)
- removed the REF** at (54.0, 71.0) (x3)
- removed the REF** at (53.0, 71.0) (x3)
- removed the REF** at (52.0, 71.0) (x3)
- removed the REF** at (51.0, 71.0) (x3)
- removed the REF** at (50.0, 71.0) (x3)
- removed the REF** at (49.0, 71.0) (x3)
- removed the REF** at (48.0, 71.0) (x3)
- removed the REF** at (47.0, 71.0) (x3)
- removed the REF** at (46.0, 71.0) (x3)
- removed the REF** at (63.0, 70.0) (x3)
- removed the REF** at (62.0, 70.0) (x3)
- removed the REF** at (61.0, 70.0) (x3)
- removed the REF** at (60.0, 70.0) (x3)
- removed the REF** at (59.0, 70.0) (x3)
- removed the REF** at (58.0, 70.0) (x3)
- removed the REF** at (57.0, 70.0) (x3)
- removed the REF** at (56.0, 70.0) (x3)
- removed the REF** at (55.0, 70.0) (x3)
- removed the REF** at (54.0, 70.0) (x3)
- removed the REF** at (53.0, 70.0) (x3)
- removed the REF** at (52.0, 70.0) (x3)
- removed the REF** at (51.0, 70.0) (x3)
- removed the REF** at (50.0, 70.0) (x3)
- removed the REF** at (49.0, 70.0) (x3)
- removed the REF** at (48.0, 70.0) (x3)
- removed the REF** at (47.0, 70.0) (x3)
- removed the REF** at (46.0, 70.0) (x3)
- removed the REF** at (63.0, 69.0) (x3)
- removed the REF** at (62.0, 69.0) (x3)
- removed the REF** at (61.0, 69.0) (x3)
- removed the REF** at (60.0, 69.0) (x3)
- removed the REF** at (59.0, 69.0) (x3)
- removed the REF** at (58.0, 69.0) (x3)
- removed the REF** at (57.0, 69.0) (x3)
- removed the REF** at (56.0, 69.0) (x3)
- removed the REF** at (55.0, 69.0) (x3)
- removed the REF** at (54.0, 69.0) (x3)
- removed the REF** at (53.0, 69.0) (x3)
- removed the REF** at (52.0, 69.0) (x3)
- removed the REF** at (51.0, 69.0) (x3)
- removed the REF** at (50.0, 69.0) (x3)
- removed the REF** at (49.0, 69.0) (x3)
- removed the REF** at (48.0, 69.0) (x3)
- removed the REF** at (47.0, 69.0) (x3)
- removed the REF** at (46.0, 69.0) (x3)
- removed the REF** at (63.0, 68.0) (x3)
- removed the REF** at (62.0, 68.0) (x3)
- removed the REF** at (61.0, 68.0) (x3)
- removed the REF** at (60.0, 68.0) (x3)
- removed the REF** at (59.0, 68.0) (x3)
- removed the REF** at (58.0, 68.0) (x3)
- removed the REF** at (57.0, 68.0) (x3)
- removed the REF** at (56.0, 68.0) (x3)
- removed the REF** at (55.0, 68.0) (x3)
- removed the REF** at (54.0, 68.0) (x3)
- removed the REF** at (53.0, 68.0) (x3)
- removed the REF** at (52.0, 68.0) (x3)
- removed the REF** at (51.0, 68.0) (x3)
- removed the REF** at (50.0, 68.0) (x3)
- removed the REF** at (49.0, 68.0) (x3)
- removed the REF** at (48.0, 68.0) (x3)
- removed the REF** at (47.0, 68.0) (x3)
- removed the REF** at (46.0, 68.0) (x3)
- removed the REF** at (63.0, 67.0) (x3)
- removed the REF** at (62.0, 67.0) (x3)
- removed the REF** at (61.0, 67.0) (x3)
- removed the REF** at (60.0, 67.0) (x3)
- removed the REF** at (59.0, 67.0) (x3)
- removed the REF** at (58.0, 67.0) (x3)
- removed the REF** at (57.0, 67.0) (x3)
- removed the REF** at (56.0, 67.0) (x3)
- removed the REF** at (55.0, 67.0) (x3)
- removed the REF** at (54.0, 67.0) (x3)
- removed the REF** at (53.0, 67.0) (x3)
- removed the REF** at (52.0, 67.0) (x3)
- removed the REF** at (51.0, 67.0) (x3)
- removed the REF** at (50.0, 67.0) (x3)
- removed the REF** at (49.0, 67.0) (x3)
- removed the REF** at (48.0, 67.0) (x3)
- removed the REF** at (47.0, 67.0) (x3)
- removed the REF** at (46.0, 67.0) (x3)
- removed the REF** at (63.0, 66.0) (x3)
- removed the REF** at (62.0, 66.0) (x3)
- removed the REF** at (61.0, 66.0) (x3)
- removed the REF** at (60.0, 66.0) (x3)
- removed the REF** at (59.0, 66.0) (x3)
- removed the REF** at (58.0, 66.0) (x3)
- removed the REF** at (57.0, 66.0) (x3)
- removed the REF** at (56.0, 66.0) (x3)
- removed the REF** at (55.0, 66.0) (x3)
- removed the REF** at (54.0, 66.0) (x3)
- removed the REF** at (53.0, 66.0) (x3)
- removed the REF** at (52.0, 66.0) (x3)
- removed the REF** at (51.0, 66.0) (x3)
- removed the REF** at (50.0, 66.0) (x3)
- removed the REF** at (49.0, 66.0) (x3)
- removed the REF** at (48.0, 66.0) (x3)
- removed the REF** at (47.0, 66.0) (x3)
- removed the REF** at (46.0, 66.0) (x3)
- removed the REF** at (63.0, 65.0) (x3)
- removed the REF** at (62.0, 65.0) (x3)
- removed the REF** at (61.0, 65.0) (x3)
- removed the REF** at (60.0, 65.0) (x3)
- removed the REF** at (59.0, 65.0) (x3)
- removed the REF** at (58.0, 65.0) (x3)
- removed the REF** at (57.0, 65.0) (x3)
- removed the REF** at (56.0, 65.0) (x3)
- removed the REF** at (55.0, 65.0) (x3)
- removed the REF** at (54.0, 65.0) (x3)
- removed the REF** at (53.0, 65.0) (x3)
- removed the REF** at (52.0, 65.0) (x3)
- removed the REF** at (51.0, 65.0) (x3)
- removed the REF** at (50.0, 65.0) (x3)
- removed the REF** at (49.0, 65.0) (x3)
- removed the REF** at (48.0, 65.0) (x3)
- removed the REF** at (47.0, 65.0) (x3)
- removed the REF** at (46.0, 65.0) (x3)
- removed the REF** at (63.0, 64.0) (x3)
- removed the REF** at (62.0, 64.0) (x3)
- removed the REF** at (61.0, 64.0) (x3)
- removed the REF** at (60.0, 64.0) (x3)
- removed the REF** at (59.0, 64.0) (x3)
- removed the REF** at (58.0, 64.0) (x3)
- removed the REF** at (57.0, 64.0) (x3)
- removed the REF** at (56.0, 64.0) (x3)
- removed the REF** at (55.0, 64.0) (x3)
- removed the REF** at (54.0, 64.0) (x3)
- removed the REF** at (53.0, 64.0) (x3)
- removed the REF** at (52.0, 64.0) (x3)
- removed the REF** at (51.0, 64.0) (x3)
- removed the REF** at (50.0, 64.0) (x3)
- removed the REF** at (49.0, 64.0) (x3)
- removed the REF** at (48.0, 64.0) (x3)
- removed the REF** at (47.0, 64.0) (x3)
- removed the REF** at (46.0, 64.0) (x3)
- removed the REF** at (63.0, 63.0) (x3)
- removed the REF** at (62.0, 63.0) (x3)
- removed the REF** at (61.0, 63.0) (x3)
- removed the REF** at (60.0, 63.0) (x3)
- removed the REF** at (59.0, 63.0) (x3)
- removed the REF** at (58.0, 63.0) (x3)
- removed the REF** at (57.0, 63.0) (x3)
- removed the REF** at (56.0, 63.0) (x3)
- removed the REF** at (55.0, 63.0) (x3)
- removed the REF** at (54.0, 63.0) (x3)
- removed the REF** at (53.0, 63.0) (x3)
- removed the REF** at (52.0, 63.0) (x3)
- removed the REF** at (51.0, 63.0) (x3)
- removed the REF** at (50.0, 63.0) (x3)
- removed the REF** at (49.0, 63.0) (x3)
- removed the REF** at (48.0, 63.0) (x3)
- removed the REF** at (47.0, 63.0) (x3)
- removed the REF** at (46.0, 63.0) (x3)
- removed the REF** at (63.0, 62.0) (x3)
- removed the REF** at (62.0, 62.0) (x3)
- removed the REF** at (61.0, 62.0) (x3)
- removed the REF** at (60.0, 62.0) (x3)
- removed the REF** at (59.0, 62.0) (x3)
- removed the REF** at (58.0, 62.0) (x3)
- removed the REF** at (57.0, 62.0) (x3)
- removed the REF** at (56.0, 62.0) (x3)
- removed the REF** at (55.0, 62.0) (x3)
- removed the REF** at (54.0, 62.0) (x3)
- removed the REF** at (53.0, 62.0) (x3)
- removed the REF** at (52.0, 62.0) (x3)
- removed the REF** at (51.0, 62.0) (x3)
- removed the REF** at (50.0, 62.0) (x3)
- removed the REF** at (49.0, 62.0) (x3)
- removed the REF** at (48.0, 62.0) (x3)
- removed the REF** at (47.0, 62.0) (x3)
- removed the REF** at (76.0, 62.0)
- removed the REF** at (46.0, 62.0)
- removed the REF** at (30.0, 62.0)
- removed the REF** at (33.0, 70.0)
- removed the REF** at (32.0, 70.0)
- removed the REF** at (31.0, 70.0)
- removed the REF** at (30.0, 70.0)
- removed the REF** at (109.0, 70.0)
- removed the REF** at (108.0, 70.0)
- removed the REF** at (107.0, 70.0)
- removed the REF** at (33.0, 69.0)
- removed the REF** at (106.0, 70.0)
- removed the REF** at (109.0, 69.0)
- removed the REF** at (108.0, 69.0)
- removed the REF** at (107.0, 69.0)
- removed the REF** at (106.0, 69.0)
- removed the REF** at (109.0, 68.0)
- removed the REF** at (108.0, 68.0)
- removed the REF** at (107.0, 68.0)
- removed the REF** at (106.0, 68.0)
- removed the REF** at (109.0, 67.0)
- removed the REF** at (32.0, 69.0)
- removed the REF** at (108.0, 67.0)
- removed the REF** at (107.0, 67.0)
- removed the REF** at (106.0, 67.0)
- removed the REF** at (109.0, 66.0)
- removed the REF** at (108.0, 66.0)
- removed the REF** at (107.0, 66.0)
- removed the REF** at (106.0, 66.0)
- removed the REF** at (109.0, 65.0)
- removed the REF** at (108.0, 65.0)
- removed the REF** at (107.0, 65.0)
- removed the REF** at (31.0, 69.0)
- removed the REF** at (106.0, 65.0)
- removed the REF** at (109.0, 64.0)
- removed the REF** at (108.0, 64.0)
- removed the REF** at (107.0, 64.0)
- removed the REF** at (106.0, 64.0)
- removed the REF** at (109.0, 63.0)
- removed the REF** at (108.0, 63.0)
- removed the REF** at (115.0, 108.0)
- removed the REF** at (107.0, 63.0)
- removed the REF** at (115.0, 107.0)
- removed the REF** at (115.0, 106.0)
- removed the REF** at (115.0, 105.0)
- removed the REF** at (106.0, 63.0)
- removed the REF** at (115.0, 104.0)
- removed the REF** at (115.0, 103.0)
- removed the REF** at (109.0, 62.0)
- removed the REF** at (115.0, 102.0)
- removed the REF** at (115.0, 101.0)
- removed the REF** at (115.0, 100.0)
- removed the REF** at (30.0, 69.0)
- removed the REF** at (108.0, 62.0)
- removed the REF** at (115.0, 99.0)
- removed the REF** at (115.0, 98.0)
- removed the REF** at (107.0, 62.0)
- removed the REF** at (115.0, 97.0)
- removed the REF** at (115.0, 96.0)
- removed the REF** at (115.0, 95.0)
- removed the REF** at (106.0, 62.0)
- removed the REF** at (115.0, 94.0)
- removed the REF** at (115.0, 93.0)
- removed the REF** at (115.0, 92.0)
- removed the REF** at (115.0, 91.0)
- removed the REF** at (115.0, 90.0)
- removed the REF** at (115.0, 89.0)
- removed the REF** at (115.0, 88.0)
- removed the REF** at (115.0, 87.0)
- removed the REF** at (115.0, 86.0)
- removed the REF** at (115.0, 85.0)
- removed the REF** at (33.0, 68.0)
- removed the REF** at (32.0, 68.0)
- removed the REF** at (31.0, 68.0)
- removed the REF** at (30.0, 68.0)
- removed the REF** at (33.0, 67.0)
- removed the REF** at (32.0, 67.0)
- removed the REF** at (31.0, 67.0)
- removed the REF** at (93.0, 70.0)
- removed the REF** at (92.0, 70.0)
- removed the REF** at (91.0, 70.0)
- removed the REF** at (90.0, 70.0)
- removed the REF** at (89.0, 70.0)
- removed the REF** at (30.0, 67.0)
- removed the REF** at (88.0, 70.0)
- removed the REF** at (87.0, 70.0)
- removed the REF** at (86.0, 70.0)
- removed the REF** at (85.0, 70.0)
- removed the REF** at (84.0, 70.0)
- removed the REF** at (83.0, 70.0)
- removed the REF** at (82.0, 70.0)
- removed the REF** at (81.0, 70.0)
- removed the REF** at (80.0, 70.0)
- removed the REF** at (79.0, 70.0)
- removed the REF** at (33.0, 66.0)
- removed the REF** at (78.0, 70.0)
- removed the REF** at (77.0, 70.0)
- removed the REF** at (76.0, 70.0)
- removed the REF** at (93.0, 69.0)
- removed the REF** at (92.0, 69.0)
- removed the REF** at (91.0, 69.0)
- removed the REF** at (90.0, 69.0)
- removed the REF** at (89.0, 69.0)
- removed the REF** at (88.0, 69.0)
- removed the REF** at (87.0, 69.0)
- removed the REF** at (32.0, 66.0)
- removed the REF** at (86.0, 69.0)
- removed the REF** at (85.0, 69.0)
- removed the REF** at (84.0, 69.0)
- removed the REF** at (83.0, 69.0)
- removed the REF** at (82.0, 69.0)
- removed the REF** at (81.0, 69.0)
- removed the REF** at (80.0, 69.0)
- removed the REF** at (79.0, 69.0)
- removed the REF** at (78.0, 69.0)
- removed the REF** at (77.0, 69.0)
- removed the REF** at (31.0, 66.0)
- removed the REF** at (76.0, 69.0)
- removed the REF** at (93.0, 68.0)
- removed the REF** at (92.0, 68.0)
- removed the REF** at (91.0, 68.0)
- removed the REF** at (90.0, 68.0)
- removed the REF** at (89.0, 68.0)
- removed the REF** at (88.0, 68.0)
- removed the REF** at (87.0, 68.0)
- removed the REF** at (86.0, 68.0)
- removed the REF** at (85.0, 68.0)
- removed the REF** at (30.0, 66.0)
- removed the REF** at (84.0, 68.0)
- removed the REF** at (83.0, 68.0)
- removed the REF** at (82.0, 68.0)
- removed the REF** at (81.0, 68.0)
- removed the REF** at (80.0, 68.0)
- removed the REF** at (79.0, 68.0)
- removed the REF** at (78.0, 68.0)
- removed the REF** at (77.0, 68.0)
- removed the REF** at (76.0, 68.0)
- removed the REF** at (93.0, 67.0)
- removed the REF** at (33.0, 65.0)
- removed the REF** at (92.0, 67.0)
- removed the REF** at (91.0, 67.0)
- removed the REF** at (90.0, 67.0)
- removed the REF** at (89.0, 67.0)
- removed the REF** at (88.0, 67.0)
- removed the REF** at (87.0, 67.0)
- removed the REF** at (86.0, 67.0)
- removed the REF** at (85.0, 67.0)
- removed the REF** at (84.0, 67.0)
- removed the REF** at (83.0, 67.0)
- removed the REF** at (32.0, 65.0)
- removed the REF** at (82.0, 67.0)
- removed the REF** at (81.0, 67.0)
- removed the REF** at (80.0, 67.0)
- removed the REF** at (79.0, 67.0)
- removed the REF** at (78.0, 67.0)
- removed the REF** at (77.0, 67.0)
- removed the REF** at (76.0, 67.0)
- removed the REF** at (93.0, 66.0)
- removed the REF** at (92.0, 66.0)
- removed the REF** at (91.0, 66.0)
- removed the REF** at (31.0, 65.0)
- removed the REF** at (90.0, 66.0)
- removed the REF** at (89.0, 66.0)
- removed the REF** at (88.0, 66.0)
- removed the REF** at (87.0, 66.0)
- removed the REF** at (86.0, 66.0)
- removed the REF** at (85.0, 66.0)
- removed the REF** at (84.0, 66.0)
- removed the REF** at (83.0, 66.0)
- removed the REF** at (82.0, 66.0)
- removed the REF** at (81.0, 66.0)
- removed the REF** at (30.0, 65.0)
- removed the REF** at (80.0, 66.0)
- removed the REF** at (79.0, 66.0)
- removed the REF** at (78.0, 66.0)
- removed the REF** at (77.0, 66.0)
- removed the REF** at (76.0, 66.0)
- removed the REF** at (93.0, 65.0)
- removed the REF** at (92.0, 65.0)
- removed the REF** at (91.0, 65.0)
- removed the REF** at (90.0, 65.0)
- removed the REF** at (89.0, 65.0)
- removed the REF** at (33.0, 64.0)
- removed the REF** at (88.0, 65.0)
- removed the REF** at (87.0, 65.0)
- removed the REF** at (86.0, 65.0)
- removed the REF** at (85.0, 65.0)
- removed the REF** at (84.0, 65.0)
- removed the REF** at (83.0, 65.0)
- removed the REF** at (82.0, 65.0)
- removed the REF** at (81.0, 65.0)
- removed the REF** at (80.0, 65.0)
- removed the REF** at (79.0, 65.0)
- removed the REF** at (32.0, 64.0)
- removed the REF** at (78.0, 65.0)
- removed the REF** at (77.0, 65.0)
- removed the REF** at (76.0, 65.0)
- removed the REF** at (93.0, 64.0)
- removed the REF** at (92.0, 64.0)
- removed the REF** at (91.0, 64.0)
- removed the REF** at (90.0, 64.0)
- removed the REF** at (89.0, 64.0)
- removed the REF** at (88.0, 64.0)
- removed the REF** at (87.0, 64.0)
- removed the REF** at (31.0, 64.0)
- removed the REF** at (86.0, 64.0)
- removed the REF** at (85.0, 64.0)
- removed the REF** at (84.0, 64.0)
- removed the REF** at (83.0, 64.0)
- removed the REF** at (82.0, 64.0)
- removed the REF** at (81.0, 64.0)
- removed the REF** at (80.0, 64.0)
- removed the REF** at (79.0, 64.0)
- removed the REF** at (78.0, 64.0)
- removed the REF** at (77.0, 64.0)
- removed the REF** at (30.0, 64.0)
- removed the REF** at (76.0, 64.0)
- removed the REF** at (93.0, 63.0)
- removed the REF** at (92.0, 63.0)
- removed the REF** at (91.0, 63.0)
- removed the REF** at (90.0, 63.0)
- removed the REF** at (89.0, 63.0)
- removed the REF** at (88.0, 63.0)
- removed the REF** at (87.0, 63.0)
- removed the REF** at (86.0, 63.0)
- removed the REF** at (85.0, 63.0)
- removed the REF** at (33.0, 63.0)
- removed the REF** at (84.0, 63.0)
- removed the REF** at (83.0, 63.0)
- removed the REF** at (82.0, 63.0)
- removed the REF** at (81.0, 63.0)
- removed the REF** at (80.0, 63.0)
- removed the REF** at (79.0, 63.0)
- removed the REF** at (78.0, 63.0)
- removed the REF** at (77.0, 63.0)
- removed the REF** at (76.0, 63.0)
- removed the REF** at (93.0, 62.0)
- removed the REF** at (32.0, 63.0)
- removed the REF** at (92.0, 62.0)
- removed the REF** at (91.0, 62.0)
- removed the REF** at (90.0, 62.0)
- removed the REF** at (89.0, 62.0)
- removed the REF** at (88.0, 62.0)
- removed the REF** at (87.0, 62.0)
- removed the REF** at (86.0, 62.0)
- removed the REF** at (85.0, 62.0)
- removed the REF** at (84.0, 62.0)
- removed the REF** at (83.0, 62.0)
- removed the REF** at (31.0, 63.0)
- removed the REF** at (82.0, 62.0)
- removed the REF** at (81.0, 62.0)
- removed the REF** at (80.0, 62.0)
- removed the REF** at (79.0, 62.0)
- removed the REF** at (78.0, 62.0)
- removed the REF** at (77.0, 62.0)
- removed the REF** at (63.0, 74.0) (x3)
- removed the REF** at (62.0, 74.0) (x3)
- removed the REF** at (61.0, 74.0) (x3)
- removed the REF** at (60.0, 74.0) (x3)
- removed the REF** at (30.0, 63.0)
- removed the REF** at (59.0, 74.0) (x3)
- removed the REF** at (58.0, 74.0) (x3)
- removed the REF** at (57.0, 74.0) (x3)
- removed the REF** at (56.0, 74.0) (x3)
- removed the REF** at (55.0, 74.0) (x3)
- removed the REF** at (54.0, 74.0) (x3)
- removed the REF** at (53.0, 74.0) (x3)
- removed the REF** at (52.0, 74.0) (x3)
- removed the REF** at (51.0, 74.0) (x3)
- removed the REF** at (50.0, 74.0) (x3)
- removed the REF** at (33.0, 62.0)
- removed the REF** at (49.0, 74.0) (x3)
- removed the REF** at (48.0, 74.0) (x3)
- removed the REF** at (47.0, 74.0) (x3)
- removed the REF** at (46.0, 74.0) (x3)
- removed the REF** at (63.0, 73.0) (x3)
- removed the REF** at (62.0, 73.0) (x3)
- removed the REF** at (61.0, 73.0) (x3)
- removed the REF** at (60.0, 73.0) (x3)
- removed the REF** at (59.0, 73.0) (x3)
- removed the REF** at (58.0, 73.0) (x3)
- removed the REF** at (32.0, 62.0)
- removed the REF** at (57.0, 73.0) (x3)
- removed the REF** at (56.0, 73.0) (x3)
- removed the REF** at (55.0, 73.0) (x3)
- removed the REF** at (54.0, 73.0) (x3)
- removed the REF** at (53.0, 73.0) (x3)
- removed the REF** at (52.0, 73.0) (x3)
- removed the REF** at (51.0, 73.0) (x3)
- removed the REF** at (50.0, 73.0) (x3)
- removed the REF** at (49.0, 73.0) (x3)
- removed the REF** at (48.0, 73.0) (x3)
- removed the REF** at (31.0, 62.0)
- removed the REF** at (47.0, 73.0) (x3)
- removed the REF** at (46.0, 73.0) (x3)
- removed the REF** at (63.0, 72.0) (x3)
- removed the REF** at (62.0, 72.0) (x3)
- removed the REF** at (61.0, 72.0) (x3)
- removed the REF** at (60.0, 72.0) (x3)
- removed the REF** at (59.0, 72.0) (x3)
- removed the REF** at (58.0, 72.0) (x3)
- removed the REF** at (57.0, 72.0) (x3)
- removed the REF** at (56.0, 72.0) (x3)
- removed the REF** at (55.0, 72.0) (x3)
- removed the REF** at (54.0, 72.0) (x3)
- removed the REF** at (53.0, 72.0) (x3)
- removed the REF** at (52.0, 72.0) (x3)
- removed the REF** at (51.0, 72.0) (x3)
- removed the REF** at (50.0, 72.0) (x3)
- removed the REF** at (49.0, 72.0) (x3)
- removed the REF** at (48.0, 72.0) (x3)
- removed the REF** at (47.0, 72.0) (x3)
- removed the REF** at (46.0, 72.0) (x3)
- removed the REF** at (63.0, 71.0) (x3)
- removed the REF** at (62.0, 71.0) (x3)
- removed the REF** at (61.0, 71.0) (x3)
- removed the REF** at (60.0, 71.0) (x3)
- added REF**: via, via:via, F.Cu at (53.0, 78.0)
- added REF**: via, via:via, F.Cu at (76.0, 26.0)
- added REF**: via, via:via, F.Cu at (64.0, 29.0)
- added REF**: via, via:via, F.Cu at (110.0, 73.0)
- added REF**: via, via:via, F.Cu at (64.0, 28.0)
- added REF**: via, via:via, F.Cu at (110.0, 72.0)
- added REF**: via, via:via, F.Cu at (64.0, 27.0)
- added REF**: via, via:via, F.Cu at (64.0, 26.0)
- added REF**: via, via:via, F.Cu at (110.0, 71.0)
- added REF**: via, via:via, F.Cu at (94.0, 74.0)
- added REF**: via, via:via, F.Cu at (94.0, 73.0)
- added REF**: via, via:via, F.Cu at (119.0, 115.0)
- added REF**: via, via:via, F.Cu at (119.0, 114.0)
- added REF**: via, via:via, F.Cu at (119.0, 113.0)
- added REF**: via, via:via, F.Cu at (119.0, 112.0)
- added REF**: via, via:via, F.Cu at (119.0, 111.0)
- added REF**: via, via:via, F.Cu at (119.0, 110.0)
- added REF**: via, via:via, F.Cu at (119.0, 109.0)
- added REF**: via, via:via, F.Cu at (119.0, 108.0)
- added REF**: via, via:via, F.Cu at (119.0, 107.0)
- added REF**: via, via:via, F.Cu at (119.0, 106.0)
- added REF**: via, via:via, F.Cu at (119.0, 105.0)
- added REF**: via, via:via, F.Cu at (119.0, 104.0)
- added REF**: via, via:via, F.Cu at (119.0, 103.0)
- added REF**: via, via:via, F.Cu at (119.0, 102.0)
- added REF**: via, via:via, F.Cu at (119.0, 101.0)
- added REF**: via, via:via, F.Cu at (119.0, 100.0)
- added REF**: via, via:via, F.Cu at (119.0, 99.0)
- added REF**: via, via:via, F.Cu at (119.0, 98.0)
- added REF**: via, via:via, F.Cu at (119.0, 97.0)
- added REF**: via, via:via, F.Cu at (119.0, 96.0)
- added REF**: via, via:via, F.Cu at (119.0, 95.0)
- added REF**: via, via:via, F.Cu at (119.0, 94.0)
- added REF**: via, via:via, F.Cu at (119.0, 93.0)
- added REF**: via, via:via, F.Cu at (119.0, 92.0)
- added REF**: via, via:via, F.Cu at (119.0, 91.0)
- added REF**: via, via:via, F.Cu at (53.0, 77.0)
- added REF**: via, via:via, F.Cu at (119.0, 90.0)
- added REF**: via, via:via, F.Cu at (119.0, 89.0)
- added REF**: via, via:via, F.Cu at (119.0, 88.0)
- added REF**: via, via:via, F.Cu at (119.0, 87.0)
- added REF**: via, via:via, F.Cu at (119.0, 86.0)
- added REF**: via, via:via, F.Cu at (119.0, 85.0)
- added REF**: via, via:via, F.Cu at (94.0, 72.0)
- added REF**: via, via:via, F.Cu at (94.0, 71.0)
- added REF**: via, via:via, F.Cu at (64.0, 74.0)
- added REF**: via, via:via, F.Cu at (63.0, 74.0)
- added REF**: via, via:via, F.Cu at (62.0, 74.0)
- added REF**: via, via:via, F.Cu at (61.0, 74.0)
- added REF**: via, via:via, F.Cu at (60.0, 74.0)
- added REF**: via, via:via, F.Cu at (59.0, 74.0)
- added REF**: via, via:via, F.Cu at (58.0, 74.0)
- added REF**: via, via:via, F.Cu at (57.0, 74.0)
- added REF**: via, via:via, F.Cu at (56.0, 74.0)
- added REF**: via, via:via, F.Cu at (94.0, 79.0)
- added REF**: via, via:via, F.Cu at (55.0, 74.0)
- added REF**: via, via:via, F.Cu at (54.0, 74.0)
- added REF**: via, via:via, F.Cu at (53.0, 74.0)
- added REF**: via, via:via, F.Cu at (52.0, 74.0)
- added REF**: via, via:via, F.Cu at (51.0, 74.0)
- added REF**: via, via:via, F.Cu at (50.0, 74.0)
- added REF**: via, via:via, F.Cu at (49.0, 74.0)
- added REF**: via, via:via, F.Cu at (48.0, 74.0)
- added REF**: via, via:via, F.Cu at (47.0, 74.0)
- added REF**: via, via:via, F.Cu at (46.0, 74.0)
- added REF**: via, via:via, F.Cu at (64.0, 73.0)
- added REF**: via, via:via, F.Cu at (63.0, 73.0)
- added REF**: via, via:via, F.Cu at (62.0, 73.0)
- added REF**: via, via:via, F.Cu at (61.0, 73.0)
- added REF**: via, via:via, F.Cu at (60.0, 73.0)
- added REF**: via, via:via, F.Cu at (59.0, 73.0)
- added REF**: via, via:via, F.Cu at (58.0, 73.0)
- added REF**: via, via:via, F.Cu at (57.0, 73.0)
- added REF**: via, via:via, F.Cu at (56.0, 73.0)
- added REF**: via, via:via, F.Cu at (55.0, 73.0)
- added REF**: via, via:via, F.Cu at (54.0, 73.0)
- added REF**: via, via:via, F.Cu at (53.0, 73.0)
- added REF**: via, via:via, F.Cu at (52.0, 73.0)
- added REF**: via, via:via, F.Cu at (51.0, 73.0)
- added REF**: via, via:via, F.Cu at (50.0, 73.0)
- added REF**: via, via:via, F.Cu at (49.0, 73.0)
- added REF**: via, via:via, F.Cu at (48.0, 73.0)
- added REF**: via, via:via, F.Cu at (47.0, 73.0)
- added REF**: via, via:via, F.Cu at (46.0, 73.0)
- added REF**: via, via:via, F.Cu at (64.0, 72.0)
- added REF**: via, via:via, F.Cu at (63.0, 72.0)
- added REF**: via, via:via, F.Cu at (62.0, 72.0)
- added REF**: via, via:via, F.Cu at (61.0, 72.0)
- added REF**: via, via:via, F.Cu at (60.0, 72.0)
- added REF**: via, via:via, F.Cu at (59.0, 72.0)
- added REF**: via, via:via, F.Cu at (58.0, 72.0)
- added REF**: via, via:via, F.Cu at (57.0, 72.0)
- added REF**: via, via:via, F.Cu at (56.0, 72.0)
- added REF**: via, via:via, F.Cu at (55.0, 72.0)
- added REF**: via, via:via, F.Cu at (54.0, 72.0)
- added REF**: via, via:via, F.Cu at (53.0, 72.0)
- added REF**: via, via:via, F.Cu at (52.0, 72.0)
- added REF**: via, via:via, F.Cu at (51.0, 72.0)
- added REF**: via, via:via, F.Cu at (50.0, 72.0)
- added REF**: via, via:via, F.Cu at (49.0, 72.0)
- added REF**: via, via:via, F.Cu at (48.0, 72.0)
- added REF**: via, via:via, F.Cu at (47.0, 72.0)
- added REF**: via, via:via, F.Cu at (46.0, 72.0)
- added REF**: via, via:via, F.Cu at (64.0, 71.0)
- added REF**: via, via:via, F.Cu at (63.0, 71.0)
- added REF**: via, via:via, F.Cu at (62.0, 71.0)
- added REF**: via, via:via, F.Cu at (61.0, 71.0)
- added REF**: via, via:via, F.Cu at (60.0, 71.0)
- added REF**: via, via:via, F.Cu at (59.0, 71.0)
- added REF**: via, via:via, F.Cu at (58.0, 71.0)
- added REF**: via, via:via, F.Cu at (57.0, 71.0)
- added REF**: via, via:via, F.Cu at (56.0, 71.0)
- added REF**: via, via:via, F.Cu at (55.0, 71.0)
- added REF**: via, via:via, F.Cu at (54.0, 71.0)
- added REF**: via, via:via, F.Cu at (53.0, 71.0)
- added REF**: via, via:via, F.Cu at (52.0, 71.0)
- added REF**: via, via:via, F.Cu at (51.0, 71.0)
- added REF**: via, via:via, F.Cu at (50.0, 71.0)
- added REF**: via, via:via, F.Cu at (49.0, 71.0)
- added REF**: via, via:via, F.Cu at (48.0, 71.0)
- added REF**: via, via:via, F.Cu at (47.0, 71.0)
- added REF**: via, via:via, F.Cu at (94.0, 78.0)
- added REF**: via, via:via, F.Cu at (34.0, 74.0)
- added REF**: via, via:via, F.Cu at (34.0, 73.0)
- added REF**: via, via:via, F.Cu at (34.0, 72.0)
- added REF**: via, via:via, F.Cu at (34.0, 71.0)
- added REF**: via, via:via, F.Cu at (53.0, 76.0)
- added REF**: via, via:via, F.Cu at (46.0, 71.0)
- added REF**: via, via:via, F.Cu at (94.0, 77.0)
- added REF**: via, via:via, F.Cu at (53.0, 79.0)
- added REF**: via, via:via, F.Cu at (94.0, 76.0)
- added REF**: via, via:via, F.Cu at (76.0, 29.0)
- added REF**: via, via:via, F.Cu at (76.0, 28.0)
- added REF**: via, via:via, F.Cu at (110.0, 74.0)
- added REF**: via, via:via, F.Cu at (76.0, 27.0)
- C1, C11, C3, C5, C7, C9: value C -> 100n
- C13: value C -> 100nC
- moved J12 6.67 mm to (34.0, 49.0)
- moved J11 5.00 mm to (33.0, 98.0)
Connections:
- J11 pad 1: +12V -> RX_BYPASS_OUT
- J11 pad 2: GND -> RX3_IN
- J11 pad 3: Xvtr_IN -> RX2_IN
- J11 pad 4: RX2_IN -> Xvtr_IN
- J11 pad 5: RX3_IN -> GND
- J11 pad 6: RX_BYPASS_OUT -> +12V
- J12 pad 1: +12V -> Ant_3
- J12 pad 2: GND -> Ant_2
- J12 pad 4: Ant_2 -> GND
- J12 pad 5: Ant_3 -> +12V
Routing:
- net GND: track 690.0 -> 854.0 mm, vias 247 -> 423
- net +12V: track 186.4 -> 225.8 mm
- net Xvtr_IN: track 55.5 -> 45.6 mm, vias 2 -> 0
- net RX_BYPASS_OUT: track 22.3 -> 28.7 mm, vias 0 -> 2
- net Ant_1: track 32.0 -> 29.0 mm
- net Ant_2: track 58.7 -> 55.9 mm, vias 0 -> 1
- net RX2_IN: track 71.6 -> 69.9 mm
- net Ant_3: track 84.1 -> 82.9 mm, vias 0 -> 1
Other:
- board text added: "+12V"
- board text removed: "+12V_In"
