File: RX_Ant.sch (KiCad schematic (older format))
At the start: 47 parts, among them J1 CONN_COAXIAL, J10 CONN_COAXIAL, J12 CONN_01X05, J13 CONN_COAXIAL, J14 Conn_01x07, J15 CONN_COAXIAL, J16 CONN_01X01, J17 CONN_01X01, J18 CONN_01X01, J19 CONN_01X01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

Commit message: upgrate to Kicad 5.0n, new up to date Gerber
Parts:
- C1, C11, C13, C2, C3, C5, C7, C9: symbol C -> RX_Ant-rescue:C
- J1, J10, J13, J15, J2, J3, J32, J37, J4, J5, J6, J8, J9: symbol CONN_COAXIAL -> RX_Ant-rescue:CONN_COAXIAL
- J12: symbol CONN_01X05 -> RX_Ant-rescue:CONN_01X05
- J14: symbol Conn_01x07 -> RX_Ant-rescue:Conn_01x07
- J16, J17, J18, J19, J20, J21, J22, J23: symbol CONN_01X01 -> RX_Ant-rescue:CONN_01X01
- L1, L2, L3, L4, L5, L6, L7, L8: symbol L_cap -> l_cap:L_cap
- RL1, RL3, RL5, RL7, RL8: symbol EC2-12NU -> ee2-5nu:EC2-12NU
- RL2, RL4, RL6: symbol Omron_G5LE -> Omron_G5LE:Omron_G5LE
Other:
- note added: "Angelia coax panel V3.0\n"
- note removed: "Angelia coax panel\n"
- moved on the sheet: J16, J17, J18, J19
